File: hydrabot.brd (EAGLE design)
At the start: 160 x 100 mm, 3 parts

Commit message: atualização de arquivos
Parts:
- removed A1: 113990105, 113990105:SEEED_113990105
- removed R1: 1k, rcl:R0805
- removed T1: (no value), transistor-neu-to92:SOT223
- added J1: USB3090-XX-X_REVE, USB3090-XX-X_REVE:GCT_USB3090-XX-X_REVE
- added SV1, SV2: (no value), gota:FE08
- added U$7: ESP32DEVKITV1, ESP32-DEVKITV1:ESP32-DEVKITV1
- added ULN2803: ULN2803AFW, ULN2803AFW:ULN2803AFW
Connections:
- removed net 3V3: A1.J1_11, A1.J2_15, A1.J2_6
- removed net DRIVER_PUMP: R1.1
- removed net N$1: R1.2, T1.1
- removed net N$2: T1.4
- removed net VIN: A1.J1_15
- new net IO13: U$7.28, ULN2803.I4
- new net IO16: U$7.6, ULN2803.I1
- new net IO17: U$7.7, ULN2803.I2
- new net IO18: U$7.9, ULN2803.I3
- new net IO25: U$7.23, ULN2803.I5
- new net IO26: U$7.24, ULN2803.I6
- new net IO27: U$7.25, ULN2803.I7
- new net IO32: U$7.21, ULN2803.I8
- new net PORTA13: SV1.1, ULN2803.O4
- new net PORTA16: SV1.7, ULN2803.O1
- new net PORTA17: SV1.5, ULN2803.O2
- new net PORTA19: SV1.3, ULN2803.O3
- new net PORTA25: SV2.7, ULN2803.O5
- new net PORTA26: SV2.5, ULN2803.O6
- new net PORTA27: SV2.3, ULN2803.O7
- new net PORTA32: SV2.1, ULN2803.O8
- new net VCC: J1.1, SV1.2, SV1.4, SV1.6, SV1.8, SV2.2, SV2.4, SV2.6, SV2.8, U$7.30, ULN2803.COMMON
- net GND: now also J1.5, J1.6, J1.7, J1.8, J1.9, U$7.2, ULN2803.GND; no longer A1.J1_10, A1.J1_14, A1.J2_14, A1.J2_7, T1.3
Routing:
- net VCC: track 0.00 -> 163.8 mm, vias 0 -> 1
- net GND: track 0.00 -> 89.0 mm, vias 0 -> 1
- net PORTA32: track 0.00 -> 45.4 mm
- net PORTA27: track 0.00 -> 42.9 mm
- net PORTA26: track 0.00 -> 39.8 mm
- net PORTA16: track 0.00 -> 39.5 mm
- net PORTA25: track 0.00 -> 36.8 mm
- net PORTA17: track 0.00 -> 36.4 mm
- net IO13: track 0.00 -> 34.2 mm, vias 0 -> 1
- net PORTA19: track 0.00 -> 32.9 mm
- net PORTA13: track 0.00 -> 30.4 mm
- net IO27: track 0.00 -> 21.8 mm, vias 0 -> 2
- net IO26: track 0.00 -> 21.5 mm, vias 0 -> 1
- net IO25: track 0.00 -> 19.5 mm
- net IO16: track 0.00 -> 19.0 mm
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- added copper zone on layer 16, net LOGO
- added copper zone on layer 1, net VCC
Other:
- board size 160 x 100 mm -> 45 x 60 mm
- board text added: "vcc"
