File: hydrabot.sch (EAGLE design)
At the start: 3 parts

Commit message: atualização de arquivos
Parts:
- removed A1: 113990105, 113990105:113990105
- removed R1: 1k, rcl:R-EU_R0805
- removed T1: (no value), transistor-neu-to92:-NPN-SOT223
- added J1: USB3090-XX-X_REVE, USB3090-XX-X_REVE:USB3090-XX-X_REVE
- added SV1, SV2: (no value), gota:FE08-1
- added U$7: ESP32DEVKITV1, ESP32-DEVKITV1:ESP32DEVKITV1
- added ULN2803: ULN2803AFW, ULN2803AFW:ULN2803AFW
Connections:
- removed net DRIVER_PUMP: R1.1
- removed net N$1: R1.2, T1.B
- removed net N$2: T1.C
- new net IO13: U$7.IO13, ULN2803.I4
- new net IO16: U$7.IO16, ULN2803.I1
- new net IO17: U$7.IO17, ULN2803.I2
- new net IO18: U$7.IO18, ULN2803.I3
- new net IO25: U$7.IO25, ULN2803.I5
- new net IO26: U$7.IO26, ULN2803.I6
- new net IO27: U$7.IO27, ULN2803.I7
- new net IO32: U$7.IO32, ULN2803.I8
- new net PORTA13: SV1.1, ULN2803.O4
- new net PORTA16: SV1.7, ULN2803.O1
- new net PORTA17: SV1.5, ULN2803.O2
- new net PORTA19: SV1.3, ULN2803.O3
- new net PORTA25: SV2.7, ULN2803.O5
- new net PORTA26: SV2.5, ULN2803.O6
- new net PORTA27: SV2.3, ULN2803.O7
- new net PORTA32: SV2.1, ULN2803.O8
- new net VCC: J1.VBUS, SV1.2, SV1.4, SV1.6, SV1.8, SV2.2, SV2.4, SV2.6, SV2.8, U$7.VIN, ULN2803.COMMON
- net GND: now also J1.SHIELD, U$7.GND, ULN2803.GND; no longer T1.E
